File: rs232/rs232/rs232.kicad_sch (KiCad schematic)
At the start: 19 parts, among them J1 Conn_01x03_Pin, J2 Conn_01x04_Pin, J3 Conn_01x03_Pin, J4 Conn_01x02_Pin

Commit message: Updated gitignore
Now ignores backup files
Parts:
- J2: footprint Connector_PinHeader_1.00mm:PinHeader_1x04_P1.00mm_Vertical -> Connector_PinHeader_2.00mm:PinHeader_1x04_P2.00mm_Vertical
Changed lines of the file:
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@@
     )
   )
-  (symbol (lib_name "Conn_01x04_Pin_1") (lib_id "Connector:Conn_01x04_Pin") (at 102.362 39.878 180) (unit 1)
+  (symbol (lib_id "Connector:Conn_01x04_Pin") (at 102.362 39.878 180) (unit 1)
     (in_bom yes) (on_board yes) (dnp no)
     (property "Reference" "J2" (at 101.6 33.274 0)
@@
       (effects (font (size 1.27 1.27)) hide)
     )
-    (property "Footprint" "Connector_PinHeader_1.00mm:PinHeader_1x04_P1.00mm_Vertical" (at 102.362 39.878 0)
+    (property "Footprint" "Connector_PinHeader_2.00mm:PinHeader_1x04_P2.00mm_Vertical" (at 102.362 39.878 0)
       (effects (font (size 1.27 1.27)) hide)
     )

Commit message: Final commit before disassociating from combined repo
Parts:
- removed J4: Conn_01x02_Pin, Connector_PinHeader_1.00mm:PinHeader_1x02_P1.00mm_Vertical, symbol Sphere:Conn_01x02_Pin
- added H1, H2, H3, H4: MountingHole_Pad, MountingHole:MountingHole_3.7mm_Pad_Via, symbol Mechanical:MountingHole_Pad
- added J2: X5 Pass Through, Package_DIP:DIP-14_W10.16mm, symbol Connector_Generic:Conn_02x07_Top_Bottom
- added J3, J4: Conn_01x03_Pin, Connector_PinHeader_2.54mm:PinHeader_1x07_P2.54mm_Vertical, symbol Connector:Conn_01x07_Pin
- E1: renamed from E99; footprint Package_DIP:DIP-6_W10.16mm -> Package_DIP:DIP-6_W7.62mm
- E30, E31: footprint Package_DIP:DIP-6_W10.16mm -> Package_DIP:DIP-6_W7.62mm
- E46: footprint Package_DIP:DIP-14_W10.16mm -> Package_DIP:DIP-14_W7.62mm
- J5: renamed from J1; footprint Connector_PinHeader_1.00mm:PinHeader_1x03_P1.00mm_Vertical -> Connector_PinHeader_2.54mm:PinHeader_1x03_P2.54mm_Vertical
- J6: renamed from J3; footprint Connector_PinHeader_1.00mm:PinHeader_1x03_P1.00mm_Vertical -> Connector_PinHeader_2.54mm:PinHeader_1x03_P2.54mm_Vertical
- J7: renamed from J2; footprint Connector_PinHeader_2.00mm:PinHeader_1x04_P2.00mm_Vertical -> Connector_PinHeader_2.54mm:PinHeader_1x04_P2.54mm_Vertical
- PB1: renamed from PB7; footprint Jumper:SolderJumper-3_P1.3mm_Open_Pad1.0x1.5mm -> Connector_PinHeader_2.54mm:PinHeader_1x03_P2.54mm_Vertical
- PB2: renamed from PB0; footprint Jumper:SolderJumper-3_P1.3mm_Open_Pad1.0x1.5mm -> Connector_PinHeader_2.54mm:PinHeader_1x03_P2.54mm_Vertical
- R16, R4, R5, R9: footprint Resistor_THT:R_Axial_DIN0204_L3.6mm_D1.6mm_P7.62mm_Horizontal -> Resistor_THT:R_Axial_DIN0414_L11.9mm_D4.5mm_P25.40mm_Horizontal
- R2: renamed from R17; footprint Resistor_THT:R_Axial_DIN0204_L3.6mm_D1.6mm_P7.62mm_Horizontal -> Resistor_THT:R_Axial_DIN0414_L11.9mm_D4.5mm_P25.40mm_Horizontal
Connections:
- net at PB2.2 (C): now also J2.2 (Pin_2), J3.6
- net at PB1.2 (C): now also J2.9 (Pin_9), J4.2
- new net: J2.7 (Pin_7), J3.1
- new net: J2.6 (Pin_6), J3.2
- new net: J2.5 (Pin_5), J3.3
- new net: J2.4 (Pin_4), J3.4
- new net: J2.3 (Pin_3), J3.5
- new net: J2.1 (Pin_1), J3.7
- new net: J2.8 (Pin_8), J4.1
- new net: J2.10 (Pin_10), J4.3
- new net: J2.11 (Pin_11), J4.4
- new net: J2.12 (Pin_12), J4.5
- new net: J2.13 (Pin_13), J4.6
- new net: J2.14 (Pin_14), J4.7
Other:
- note added: "(E40)"
- note added: "* The original schematic separates chip pins out for ease of diagramming. This version does not."
- note added: "B XX-XXX-2024 A. Shapton Updated after first board production: * integrated E40 functionality on PCB * Updated footprints * Used connectors instead of pins * Altered schematic layout for clarity"
- note added: "To X5"
- note added: "©2024"
- note removed: "* The original schematic separates chip pins out for ease of diagramming. This version does not"
- note removed: "0.2 XX-XXX-2023 A. Shapton Updated after first board production: * integrated E40 functionality on PCB"
- note removed: "©2023"
- moved on the sheet: C12, D10, D11, E1, E30, E31, E46, E52, J5, J6, J7, PB1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
